File: Power.kicad_sch (KiCad schematic)
At the start: 86 parts, among them U3 TPS54226PWPRPWP14_2P31X2P46-L

Commit message: Update V0.3
Quashed all the DRC errors! Probably pretty stable now.
Parts:
- C1: footprint (none) -> oresat-proto-card:.0805-B-NOSILK
- C17, C22, C23, C3, R17, R24, R3, R39, R40, R45, R46, R52, R53, R54, R55, R56, R57, R58, R59, R60, R61, R62, R63, R65, R66, R67, R68, R69, R70, R71, R72, R73, R76, R77, R78, R79, R80, R81, R82, R83: footprint (none) -> oresat-proto-card:.0603-C-NOSILK
- C8: value (none) -> 1u; footprint (none) -> oresat-proto-card:.0603-C-NOSILK
- D3, D6, D7: footprint (none) -> oresat-proto-card:LED-0603
- Q1, Q2, Q7: footprint (none) -> oresat-proto-card:SOT23-6
- Q8, Q9: footprint (none) -> oresat-proto-card:SOT23
- R64: footprint (none) -> oresat-proto-card:R1206
- TP15, TP2, TP21, TP23, TP24, TP31, TP32, TP33, TP34, TP35, TP36, TP37, TP38, TP39, TP4, TP40, TP41, TP42: value (none) -> TEST-POINT-LARGE-SQUARE; footprint (none) -> oresat-proto-card:1X01
- U11, U12: value (none) -> MIC842LYC5; footprint (none) -> oresat-proto-card:SC70-5
- U2, U6: footprint (none) -> oresat-proto-card:QFN65P400X400X80-17T210
