File: Power.kicad_sch (KiCad schematic)
At the start: 86 parts, among them U3 TPS54226PWPRPWP14_2P31X2P46-L

Commit message: Updated card
Parts:
- removed TP32: (no value), symbol oresat-proto-card-eagle-import:TEST-POINT-LARGE-SQUARE
- C1: footprint (none) -> oresat-proto-card:.0805-B-NOSILK
- C17, C22, C23, C3, R17, R24, R3, R39, R40, R45, R46, R52, R53, R54, R55, R56, R57, R58, R59, R60, R61, R62, R63, R65, R66, R67, R68, R69, R70, R71, R72, R73, R76, R77, R78, R79, R80, R81, R82, R83: footprint (none) -> oresat-proto-card:.0603-C-NOSILK
- C8: value (none) -> 1u; footprint (none) -> oresat-proto-card:.0603-C-NOSILK
- D3, D6, D7: footprint (none) -> oresat-proto-card:LED-0603
- Q1, Q2, Q7: footprint (none) -> oresat-proto-card:SOT23-6
- Q8, Q9: footprint (none) -> oresat-proto-card:SOT23
- R64: footprint (none) -> oresat-proto-card:R1206
- TP15, TP2, TP21, TP23, TP24, TP31, TP33, TP34, TP35, TP36, TP37, TP38, TP39, TP4, TP40, TP41, TP42: value (none) -> TEST-POINT-LARGE-SQUARE; footprint (none) -> oresat-proto-card:1X01
- U11, U12: value (none) -> MIC842LYC5; footprint (none) -> oresat-proto-card:SC70-5
- U2, U6: footprint (none) -> oresat-proto-card:QFN65P400X400X80-17T210

Commit message: Reverted All Changes to V0.3
Parts:
- added TP32: TEST-POINT-LARGE-SQUARE, oresat-proto-card:1X01, symbol oresat-proto-card-eagle-import:TEST-POINT-LARGE-SQUARE
Changed lines of the file:
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@@
+    (stroke (width 0) (type default) (color 0 0 0 0))
+  )
+  (wire (pts (xy 417.83 233.68) (xy 422.91 233.68))
     (stroke (width 0) (type default) (color 0 0 0 0))
   )
@@
       (effects (font (size 1.778 1.5113)) (justify left bottom) hide)
     )
+    (pin "1")
+    (pin "5")
+    (pin "6")
     (pin "2")
     (pin "3")
@@
     (pin "5")
     (pin "6")
+    (pin "2")
+    (pin "3")
+    (pin "4")
   )
   (symbol (lib_id "oresat-proto-card-eagle-import:VBUSP") (at 378.46 190.5 0) (unit 1)
@@
     (pin "5")
     (pin "6")
+    (pin "2")
+    (pin "3")
+    (pin "4")
   )
   (symbol (lib_id "oresat-proto-card-eagle-import:GND") (at 129.54 260.35 0) (unit 1)
@@
     (pin "5")
     (pin "6")
+    (pin "2")
+    (pin "3")
+    (pin "4")
   )
   (symbol (lib_id "oresat-proto-card-eagle-import:GND") (at 243.586 105.156 0) (mirror y) (unit 1)
@@
     (pin "2")
   )
+  (symbol (lib_id "oresat-proto-card-eagle-import:TEST-POINT-LARGE-SQUARE") (at 422.91 233.68 0) (unit 1)
+    (in_bom yes) (on_board yes)
+    (property "Reference" "TP32" (id 0) (at 419.1 237.49 0)
+      (effects (font (size 1.27 1.0795)) (justify left bottom))
+    )
+    (property "Value" "TEST-POINT-LARGE-SQUARE" (id 1) (at 422.91 233.68 0)
+      (effects (font (size 1.27 1.27)) hide)
+    )
+    (property "Footprint" "oresat-proto-card:1X01" (id 2) (at 422.91 233.68 0)
+      (effects (font (size 1.27 1.27)) hide)
+    )
+    (property "Datasheet" "" (id 3) (at 422.91 233.68 0)
+      (effects (font (size 1.27 1.27)) hide)
+    )
+    (pin "1")
+  )
   (symbol (lib_id "oresat-proto-card-eagle-import:TEST-POINT-LARGE-SQUARE") (at 414.02 195.58 0) (unit 1)

Commit message: V0.4 BOM Updates and Footprint Fixes
Parts:
- Q1: Generic (none) -> N; Manufacturer_Name (none) -> Diodes Incorporated; Manufacturer_Part_Number (none) -> DMP2240UDM-7
- Q2, Q7: Generic (none) -> N; Manufacturer_Name (none) -> Diodes Incorporated; Manufacturer_Part_Number (none) -> DMP3050LVT-7; Notes (none) -> Make sure to verify footprint
- Q8, Q9: Generic (none) -> N; Manufacturer_Name (none) -> Microchip Technology; Manufacturer_Part_Number (none) -> PMV45EN2R
- U11, U12: Generic (none) -> N; Manufacturer_Name (none) -> Microchip Technology; Manufacturer_Part_Number (none) -> MIC842LYC5-TR
- U2: Generic (none) -> N; Manufacturer_Name (none) -> Maxim; Manufacturer_Part_Number (none) -> MAX7310ATE+
- U6: Generic (none) -> N; Manufacturer_Name (none) -> Maxim; Manufacturer_Part_Number (none) -> MAX4211FETE+
