File: Microcontroller.kicad_sch (KiCad schematic)
At the start: 25 parts

Commit message: Update V0.3
Quashed all the DRC errors! Probably pretty stable now.
Parts:
- C13, C14, C15, C18, C19, C20, C21, R47, R48, R49, R50, R51: footprint (none) -> oresat-proto-card:.0603-C-NOSILK
- D5: footprint (none) -> oresat-proto-card:LED-0603
- J7: value (none) -> ORESAT-DEBUG-CONNECTOR-ALL; footprint (none) -> oresat-proto-card:TE_2-1734592-0
- JP11, JP8: footprint (none) -> oresat-proto-card:2X10
- TP25, TP26, TP27, TP28, TP29, TP30: value (none) -> TEST-POINT-LARGE-SQUARE; footprint (none) -> oresat-proto-card:1X01
- U1: footprint (none) -> oresat-proto-card:SOT23-8_TI-DCN
- U7: footprint (none) -> oresat-proto-card:STM32F091C
- X2: footprint (none) -> oresat-proto-card:CRYSTAL_2.5X2

Commit message: V0.4 BOM Updates and Footprint Fixes
Parts:
- J7: Manufacturer_Name (none) -> TE Connectivity AMP Connectors; Manufacturer_Part_Number (none) -> 2-1734592-0
- U1: Generic (none) -> N; Manufacturer_Part_Number (none) -> TCAN330GDCNT
- U7: Generic (none) -> N; Manufacturer_Name (none) -> ST Microelectronics; Manufacturer_Part_Number (none) -> STM32F091CCT6
- X2: Generic (none) -> Y; Manufacturer_Part_Number (none) -> ECS-160-10-36Q-ES-TR
Changed lines of the file:
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@@
+      (effects (font (size 1.27 1.27)) hide)
+    )
+    (property "Manufacturer_Part_Number" "2-1734592-0" (id 4) (at 38.1 226.06 0)
+      (effects (font (size 1.27 1.27)) hide)
+    )
+    (property "Manufacturer_Name" "TE Connectivity AMP Connectors" (id 5) (at 38.1 226.06 0)
+      (effects (font (size 1.27 1.27)) hide)
+    )
+    (property "Description" "20 Position FPC Connector Contacts, Bottom 0.020\" (0.50mm) Surface Mount, Right Angle" (id 6) (at 38.1 226.06 0)
       (effects (font (size 1.27 1.27)) hide)
     )
@@
       (effects (font (size 1.778 1.5113)) (justify left bottom) hide)
     )
+    (property "Manufacturer_Part_Number" "ECS-160-10-36Q-ES-TR" (id 5) (at 81.28 101.6 90)
+      (effects (font (size 1.27 1.27)) hide)
+    )
+    (property "Description" "16MHz ±30ppm Crystal 10pF 80 Ohms" (id 6) (at 81.28 101.6 90)
+      (effects (font (size 1.27 1.27)) hide)
+    )
+    (property "Generic" "Y" (id 7) (at 81.28 101.6 90)
+      (effects (font (size 1.27 1.27)) hide)
+    )
     (pin "1")
     (pin "2")
@@
     (property "Value" "" (id 4) (at 411.48 137.16 0)
       (effects (font (size 1.778 1.5113)) (justify left bottom) hide)
+    )
+    (property "Manufacturer_Part_Number" "TCAN330GDCNT" (id 5) (at 411.48 137.16 0)
+      (effects (font (size 1.27 1.27)) hide)
+    )
+    (property "Description" "Transceiver CANbus SOT-23-8" (id 6) (at 411.48 137.16 0)
+      (effects (font (size 1.27 1.27)) hide)
+    )
+    (property "Generic" "N" (id 7) (at 411.48 137.16 0)
+      (effects (font (size 1.27 1.27)) hide)
     )
     (pin "1")
@@
       (effects (font (size 1.27 1.27)) hide)
     )
-    (property "Datasheet" "" (id 3) (at 236.22 116.84 0)
+    (property "Datasheet" "https://www.st.com/content/ccc/resource/technical/document/datasheet/95/3c/2e/5b/21/09/45/a6/DM00115237.pdf/files/DM00115237.pdf/jcr:content/translations/en.DM00115237.pdf" (id 3) (at 236.22 116.84 0)
       (effects (font (size 1.27 1.27)) hide)
     )
@@
       (effects (font (size 1.778 1.5113)) (justify left bottom) hide)
     )
-    (pin "1")
+    (property "Generic" "N" (id 5) (at 236.22 116.84 0)
+      (effects (font (size 1.27 1.27)) hide)
+    )
+    (property "Manufacturer_Part_Number" "STM32F091CCT6" (id 6) (at 236.22 116.84 0)
+      (effects (font (size 1.27 1.27)) hide)
+    )
+    (property "Manufacturer_Name" "ST Microelectronics" (id 7) (at 236.22 116.84 0)
+      (effects (font (size 1.27 1.27)) hide)
+    )
+    (pin "1")
